File: pcb/ephys-test-module-32.kicad_sch (KiCad schematic)
At the start: 1 part

Commit message: Libraries links updated
Removed local Libraries from Project
. KiCAD libraries
. open-ephys kicad library
. jonnew library

Created new manufacturing files
Parts:
- H1: footprint _footprint Lib:OEPS_SN-STICKER-8x20mm -> open-ephys:OEPS_SN-STICKER-8x20mm; symbol _symbol Lib:OEPS-SN -> open-ephys:OEPS-SN; now in the parts list
Changed lines of the file:
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@@
 	)
 	(symbol
-		(lib_id "_symbol Lib:OEPS-SN")
+		(lib_id "open-ephys:OEPS-SN")
 		(at 271.78 165.1 0)
 		(unit 1)
 		(exclude_from_sim no)
-		(in_bom no)
+		(in_bom yes)
 		(on_board yes)
 		(dnp no)
@@
 			)
 		)
-		(property "Footprint" "_footprint Lib:OEPS_SN-STICKER-8x20mm"
+		(property "Footprint" "open-ephys:OEPS_SN-STICKER-8x20mm"
 			(at 271.78 165.1 0)
 			(effects
